Commit message: Add gripper

File: lynx2.urdf (robot description, URDF)
Before this commit: robot lynxmotion_AL5D, 9 links, 9 joints
Links:
- removed link effector
- added link lbr_iiwa_with_wsg50__base_link, mass 0.2; collision box size=0.05 0.05 0.1; visual box size=0.05 0.05 0.1
- added link lbr_iiwa_with_wsg50__left_finger, mass 0.2; collision box size=0.01 0.01 0.08; visual box size=0.01 0.01 0.08
- added link lbr_iiwa_with_wsg50__left_finger_base, mass 0.2; collision mesh filename=meshes/finger_base_left.stl scale=1 1 1; visual mesh filename=meshes/finger_base_left.stl scale=1 1 1
- added link lbr_iiwa_with_wsg50__left_finger_tip, mass 0.2; collision mesh filename=meshes/finger_tip_left.stl scale=1 1 1; visual mesh filename=meshes/finger_tip_left.stl scale=1 1 1
- added link lbr_iiwa_with_wsg50__right_finger, mass 0.2; collision box size=0.01 0.01 0.08; visual box size=0.01 0.01 0.08
- added link lbr_iiwa_with_wsg50__right_finger_base, mass 0.2; collision mesh filename=meshes/finger_base_right.stl scale=1 1 1; visual mesh filename=meshes/finger_base_right.stl scale=1 1 1
- added link lbr_iiwa_with_wsg50__right_finger_tip, mass 0.2; collision mesh filename=meshes/finger_tip_right.stl scale=1 1 1; visual mesh filename=meshes/finger_tip_right.stl scale=1 1 1
Joints:
- removed joint effector_joint
- added joint lbr_iiwa_with_wsg50__base_left_finger_joint: type revolute, parent lbr_iiwa_with_wsg50__base_link, child lbr_iiwa_with_wsg50__left_finger, origin xyz=0     0.024  0.045 rpy=0   -0.05  0, axis 0  1  0, limit lower=-10.4 upper=10.01 effort=100.0 velocity=0.0
- added joint lbr_iiwa_with_wsg50__base_right_finger_joint: type revolute, parent lbr_iiwa_with_wsg50__base_link, child lbr_iiwa_with_wsg50__right_finger, origin xyz=0     0.024  0.045 rpy=0    0.05  0, axis 0  1  0, limit lower=-10.01 upper=10.4 effort=100.0 velocity=0.0
- added joint lbr_iiwa_with_wsg50__left_base_tip_joint: type revolute, parent lbr_iiwa_with_wsg50__left_finger_base, child lbr_iiwa_with_wsg50__left_finger_tip, origin xyz=0.0034   0       0.06175 rpy=0   0.5  0, axis 0  1  0, limit lower=-10.1 upper=10.3 effort=0.0 velocity=0.0
- added joint lbr_iiwa_with_wsg50__left_finger_base_joint: type fixed, parent lbr_iiwa_with_wsg50__left_finger, child lbr_iiwa_with_wsg50__left_finger_base, origin xyz=-0.00099  0       0.08015 rpy=0   -0.25  0, axis 0  0  0, limit lower=0 upper=0 effort=0 velocity=0
- added joint lbr_iiwa_with_wsg50__right_base_tip_joint: type revolute, parent lbr_iiwa_with_wsg50__right_finger_base, child lbr_iiwa_with_wsg50__right_finger_tip, origin xyz=-0.0034   0       0.06175 rpy=0  -0.5  0, axis 0  1  0, limit lower=-10.3 upper=10.1 effort=0.0 velocity=0.0
- added joint lbr_iiwa_with_wsg50__right_finger_base_joint: type fixed, parent lbr_iiwa_with_wsg50__right_finger, child lbr_iiwa_with_wsg50__right_finger_base, origin xyz=0.00099  0       0.08015 rpy=0    0.25  0, axis 0  0  0, limit lower=0 upper=0 effort=0 velocity=0
- joint servo5: child effector -> lbr_iiwa_with_wsg50__base_link

Commit message: env ready for training

File: lynx2.urdf (robot description, URDF)
Before this commit: robot lynxmotion_AL5D, 15 links, 14 joints
Links:
- removed link lbr_iiwa_with_wsg50__base_link
- removed link lbr_iiwa_with_wsg50__left_finger
- removed link lbr_iiwa_with_wsg50__left_finger_base
- removed link lbr_iiwa_with_wsg50__left_finger_tip
- removed link lbr_iiwa_with_wsg50__right_finger
- removed link lbr_iiwa_with_wsg50__right_finger_base
- removed link lbr_iiwa_with_wsg50__right_finger_tip
- added link down_finger; collision box size=0.02 0.028575 0.01; visual box size=0.02 0.028575 0.01
- added link effector_base_link; collision box size=0.04 0.0422 0.09; visual box size=0.04 0.0422 0.09
- added link up_finger; collision box size=0.02 0.028575 0.01; visual box size=0.02 0.028575 0.01
- link base_link: mass None -> 100000
- link first_servo_h: geometry collision cylinder length=0.05 radius=0.02; visual cylinder length=0.05 radius=0.02
- link second_servo_h: geometry collision cylinder length=0.05 radius=0.02; visual cylinder length=0.05 radius=0.02
- link third_servo_h: geometry collision cylinder length=0.05 radius=0.02; visual cylinder length=0.05 radius=0.02
Joints:
- removed joint lbr_iiwa_with_wsg50__base_left_finger_joint
- removed joint lbr_iiwa_with_wsg50__base_right_finger_joint
- removed joint lbr_iiwa_with_wsg50__left_base_tip_joint
- removed joint lbr_iiwa_with_wsg50__left_finger_base_joint
- removed joint lbr_iiwa_with_wsg50__right_base_tip_joint
- removed joint lbr_iiwa_with_wsg50__right_finger_base_joint
- removed joint servo2_to_base
- added joint base_to_robot: type fixed, parent base_link, child first_link, origin xyz=0 0 0.025
- added joint gripper_down: type prismatic, parent effector_base_link, child down_finger, origin xyz=0 0 0, axis 0 0 1, limit lower=-0.015 upper=0.03 effort=1000.0 velocity=0.5
- added joint gripper_up: type prismatic, parent effector_base_link, child up_finger, origin xyz=0 0 0, axis 0 0 -1, limit lower=-0.015 upper=0.03 effort=1000.0 velocity=0.5
- joint servo1: axis (none) -> 0 0 1; child first_link -> first_servo_h; limit (none) -> lower=-1.4 upper=1.4 effort=1000.0 velocity=0.5; origin xyz=0 0 0.025 -> xyz=0 0 0.0562; parent base_link -> first_link; type fixed -> revolute
- joint servo2: limit lower=0.0 upper=3.14159 effort=1000.0 velocity=0.5 -> lower=-1.2 upper=1.4 effort=1000.0 velocity=0.5
- joint servo3: limit lower=0.0 upper=3.14159 effort=1000.0 velocity=0.5 -> lower=-1.8 upper=1.7 effort=1000.0 velocity=0.5
- joint servo4: limit lower=0.0 upper=3.14159 effort=1000.0 velocity=0.5 -> lower=-1.9 upper=1.7 effort=1000.0 velocity=0.5
- joint servo5: child lbr_iiwa_with_wsg50__base_link -> effector_base_link; limit lower=0.0 upper=3.14159 effort=1000.0 velocity=0.5 -> lower=-2.0 upper=1.5 effort=1000.0 velocity=0.5
